File: PCB_NiMH_Charger_Tester.kicad_sch (KiCad schematic)
At the start: 63 parts, among them J1 USB_C_Receptacle_PowerOnly_6P, J2 USB_C_Receptacle_USB2.0_16P, J3 UPDI v2 header, J4 SSD1306, J5 Serial Header, Q1 DTC114EL, Q2 DTA114EL, Q3 MTB060P06I3, Q4 MTA100N10KRI3, SW1 SW_Push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

Commit message: Connect Vchg/Vdis to AVR
Also, change J3/J5 direction.
Connections:
- net Vdis: now reaches Q4.3 (S), R15.2, R18.1, TP3.1
- net Vdis: now also U1.17 (XTAL32K2/PF1)
- net Vchg: now reaches U1.16 (XTAL32K1/PF0)
- net Vchg: now also Q3.3 (S), R12.2, R17.2, TP2.1
- no-connect marks 13 -> 11
Changed lines of the file:
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@@
 	(title_block
 		(title "NiMH Charger & Tester")
-		(date "2025-09-05")
+		(date "2025-09-26")
 		(rev "2")
 		(company "K.Takata")
@@
 	)
 	(junction
+		(at 191.77 100.33)
+		(diameter 0)
+		(color 0 0 0 0)
+	)
+	(junction
 		(at 135.89 156.21)
 		(diameter 0)
@@
 	(junction
 		(at 50.8 25.4)
+		(diameter 0)
+		(color 0 0 0 0)
+	)
+	(junction
+		(at 191.77 144.78)
 		(diameter 0)
 		(color 0 0 0 0)
@@
 	)
 	(no_connect
-		(at 29.21 119.38)
-	)
-	(no_connect
 		(at 273.05 38.1)
 	)
@@
 		(at 44.45 95.25)
 	)
-	(no_connect
-		(at 29.21 121.92)
-	)
 	(wire
 		(pts
@@
 	(wire
 		(pts
+			(xy 200.66 144.78) (xy 191.77 144.78)
+		)
+		(stroke
+			(width 0)
+			(type default)
+		)
+	)
+	(wire
+		(pts
 			(xy 148.59 96.52) (xy 151.13 96.52)
 		)
@@
 		(pts
 			(xy 160.02 118.11) (xy 157.48 118.11)
+		)
+		(stroke
+			(width 0)
+			(type default)
+		)
+	)
+	(wire
+		(pts
+			(xy 200.66 100.33) (xy 191.77 100.33)
 		)
 		(stroke
@@
 		)
 	)
+	(global_label "Vdis"
+		(shape output)
+		(at 200.66 144.78 0)
+		(fields_autoplaced yes)
+		(effects
+			(font
+				(size 1.27 1.27)
+			)
+			(justify left)
+		)
+		(property "Intersheetrefs" "${INTERSHEET_REFS}"
+			(at 207.5157 144.78 0)
+			(effects
+				(font
+					(size 1.27 1.27)
+				)
+				(justify left)
+				(hide yes)
+			)
+		)
+	)
 	(global_label "TX"
 		(shape output)
@@
 		)
 	)
+	(global_label "Vdis"
+		(shape input)
+		(at 29.21 121.92 180)
+		(fields_autoplaced yes)
+		(effects
+			(font
+				(size 1.27 1.27)
+			)
+			(justify right)
+		)
+		(property "Intersheetrefs" "${INTERSHEET_REFS}"
+			(at 22.3543 121.92 0)
+			(effects
+				(font
+					(size 1.27 1.27)
+				)
+				(justify right)
+				(hide yes)
+			)
+		)
+	)
 	(global_label "Vbt1"
 		(shape output)
@@
 		)
 	)
+	(global_label "Vchg"
+		(shape output)
+		(at 200.66 100.33 0)
+		(fields_autoplaced yes)
+		(effects
+			(font
+				(size 1.27 1.27)
+			)
+			(justify left)
+		)
+		(property "Intersheetrefs" "${INTERSHEET_REFS}"
+			(at 208.1204 100.33 0)
+			(effects
+				(font
+					(size 1.27 1.27)
+				)
+				(justify left)
+				(hide yes)
+			)
+		)
+	)
 	(global_label "PWMdis"
 		(shape input)
@@
 				(hide yes)
 			)
+		)
+	)
+	(global_label "Vchg"
+		(shape input)
+		(at 29.21 119.38 180)
+		(fields_autoplaced yes)
+		(effects
+			(font
+				(size 1.27 1.27)
+			)
+			(justify right)
+		)
+		(property "Intersheetrefs" "${INTERSHEET_REFS}"
+			(at 21.7496 119.38 0)
+			(effects
+				(font
+					(size 1.27 1.27)
+				)
+				(justify right)
+				(hide yes)
+			)
